Commit message: footprint origin

File: urdf/vector.xacro (robot description, xacro)
@@ -5,5 +5,5 @@
   <link name="base_footprint"/>
   <joint name="base_footprint_joint" type="fixed">
-    <origin rpy="0 0 0" xyz="0 0 0.027"/>
+    <origin rpy="0 0 0" xyz="-0.01 0 0.027"/>
     <parent link="base_footprint"/>
     <child link="base_link"/>
